File: KiCAD/Test_Design/Test_Design.kicad_sch (KiCad schematic)
At the start: 0 parts

Commit message: made a circuit
battery and resistor
Parts:
- added BT1: Battery_Cell, symbol Device:Battery_Cell
- added R1: R, symbol Device:R
Connections:
- new net: BT1.1 (+), R1.1
- new net: BT1.2 (-), R1.2
